Commit message: rename link_* -> J*
the workaround is done to avoid conflict from stower robot

File: denso_robot_descriptions/vs068a4av6w4n_description/urdf/vs068a4av6w4n.xacro (robot description, xacro)
@@ -7,7 +7,7 @@
       <xacro:insert_block name="origin"/>
       <parent link="${parent}"/>
-      <child link="link_0"/>
+      <child link="J0"/>
     </joint>
-    <link name="link_0">
+    <link name="J0">
       <visual>
 	<geometry>
@@ -27,6 +27,6 @@
     </link>
     <joint name="joint_1" type="revolute">
-      <parent link="link_0" />
-      <child link="link_1" />
+      <parent link="J0" />
+      <child link="J1" />
       <origin xyz="0 0 0.164" rpy="0 0 0"/>
       <axis xyz="0 0 1" />
@@ -34,5 +34,5 @@
       <dynamics damping="0" friction="0" />
     </joint>
-    <link name="link_1">
+    <link name="J1">
       <visual>
 	<geometry>
@@ -52,6 +52,6 @@
     </link>
     <joint name="joint_2" type="revolute">
-      <parent link="link_1" />
-      <child link="link_2" />
+      <parent link="J1" />
+      <child link="J2" />
       <origin xyz="0.03 0.0 0.1975" rpy="0 0 0"/>
       <axis xyz="0 1 0" />
@@ -59,5 +59,5 @@
       <dynamics damping="0" friction="0" />
     </joint>
-    <link name="link_2">
+    <link name="J2">
       <visual>
 	<geometry>
@@ -77,6 +77,6 @@
     </link>
     <joint name="joint_3" type="revolute">
-      <parent link="link_2" />
-      <child link="link_3" />
+      <parent link="J2" />
+      <child link="J3" />
       <origin xyz="0.0 0.0 0.340" rpy="0 0 0"/>
       <axis xyz="0 1 0" />
@@ -84,5 +84,5 @@
       <dynamics damping="0" friction="0" />
     </joint>
-    <link name="link_3">
+    <link name="J3">
       <visual>
 	<geometry>
@@ -102,6 +102,6 @@
     </link>
     <joint name="joint_4" type="revolute">
-      <parent link="link_3" />
-      <child link="link_4" />
+      <parent link="J3" />
+      <child link="J4" />
       <origin xyz="-0.020 0.000 0.197" rpy="0 0 0"/>
       <axis xyz="0 0 1" />
@@ -109,5 +109,5 @@
       <dynamics damping="0" friction="0" />
     </joint>
-    <link name="link_4">
+    <link name="J4">
       <visual>
 	<geometry>
@@ -127,6 +127,6 @@
     </link>
     <joint name="joint_5" type="revolute">
-      <parent link="link_4" />
-      <child link="link_5" />
+      <parent link="J4" />
+      <child link="J5" />
       <origin xyz="0.0 0.0 0.143" rpy="0 0 0"/>
       <axis xyz="0 1 0" />
@@ -134,5 +134,5 @@
       <dynamics damping="0" friction="0" />
     </joint>
-    <link name="link_5">
+    <link name="J5">
       <visual>
 	<geometry>
@@ -152,6 +152,6 @@
     </link>
     <joint name="joint_6" type="revolute">
-      <parent link="link_5" />
-      <child link="link_6" />
+      <parent link="J5" />
+      <child link="J6" />
       <origin xyz="0.0 0.0 0.08" rpy="0 0 0"/>
       <axis xyz="0 0 1" />
@@ -159,5 +159,5 @@
       <dynamics damping="0" friction="0" />
     </joint>
-    <link name="link_6">
+    <link name="J6">
       <inertial>
 	<mass value="1" />
